Commit message: Added roller to rover chassis

File: rorover_skid_steer/urdf/rover_fixed_skid.urdf (robot description, URDF)
Before this commit: robot RoRoverDiff, 14 links, 13 joints
Links:
- added link roller, mass 0.768; collision mesh filename=package://rorover_skid_steer/meshes/Rover_Roller.stl; visual mesh filename=package://rorover_skid_steer/meshes/Rover_Roller.stl
- link chassis: mass 5.306 -> 9.244
Joints:
- added joint roller_joint: type continuous, parent chassis, child roller, origin xyz=-0.330 0.0 0.0 rpy=0.0 0.0 0.0, axis 0 1 0
